File: miniboard-opamp.sch (KiCad schematic (older format))
At the start: 0 parts

Commit message: Start routing
Parts:
- added C1, C2: 330n, Capacitors_SMD:C_0603_HandSoldering, symbol C_Small
- added C3, C4: 100n, Capacitors_SMD:C_0603_HandSoldering, symbol C_Small
- added P1, P3, P4: CONN_01X03, Socket_Strips:Socket_Strip_Straight_1x03, symbol CONN_01X03
- added R1, R10, R11, R12, R2, R3, R4, R5, R6, R7, R8, R9: R, Resistors_SMD:R_0603_HandSoldering, symbol R
- added U1: L78L12, TO_SOT_Packages_SMD:SOT89-3_Housing, symbol L78L12
- added U2: L79L12, TO_SOT_Packages_SMD:SOT89-3_Housing, symbol L79L12
- added U3: TL072, Housings_SOIC:SOIC-8_3.9x4.9mm_Pitch1.27mm, symbol TL072
Connections:
- net labels added: -12_filter, 12_filter, GND
- wire segments 0 -> 60
