File: miniboard-opamp.sch (KiCad schematic (older format))
At the start: 22 parts, among them P1 CONN_01X03, P3 CONN_01X03, P4 CONN_01X03, U1 L78L12, U2 L79L12, U3 TL072

Commit message: 1st version finished
Parts:
- R1, R10, R11, R12, R2, R3, R4, R5, R6, R7, R8, R9: footprint Resistors_SMD:R_0603_HandSoldering -> pad:R_0603_nodraw
Changed lines of the file:
@@
 F 0 "R2" V 6830 2500 50  0000 C CNN
 F 1 "R" V 6750 2500 50  0000 C CNN
-F 2 "Resistors_SMD:R_0603_HandSoldering" V 6680 2500 30  0001 C CNN
+F 2 "pad:R_0603_nodraw" V 6680 2500 30  0001 C CNN
 F 3 "" H 6750 2500 30  0000 C CNN
 	1    6750 2500
@@
 F 0 "R1" V 6830 2300 50  0000 C CNN
 F 1 "R" V 6750 2300 50  0000 C CNN
-F 2 "Resistors_SMD:R_0603_HandSoldering" V 6680 2300 30  0001 C CNN
+F 2 "pad:R_0603_nodraw" V 6680 2300 30  0001 C CNN
 F 3 "" H 6750 2300 30  0000 C CNN
 	1    6750 2300
@@
 F 0 "R5" V 7930 3100 50  0000 C CNN
 F 1 "R" V 7850 3100 50  0000 C CNN
-F 2 "Resistors_SMD:R_0603_HandSoldering" V 7780 3100 30  0001 C CNN
+F 2 "pad:R_0603_nodraw" V 7780 3100 30  0001 C CNN
 F 3 "" H 7850 3100 30  0000 C CNN
 	1    7850 3100
@@
 F 0 "R4" V 7180 2750 50  0000 C CNN
 F 1 "R" V 7100 2750 50  0000 C CNN
-F 2 "Resistors_SMD:R_0603_HandSoldering" V 7030 2750 30  0001 C CNN
+F 2 "pad:R_0603_nodraw" V 7030 2750 30  0001 C CNN
 F 3 "" H 7100 2750 30  0000 C CNN
 	1    7100 2750
@@
 F 0 "R3" V 7180 1800 50  0000 C CNN
 F 1 "R" V 7100 1800 50  0000 C CNN
-F 2 "Resistors_SMD:R_0603_HandSoldering" V 7030 1800 30  0001 C CNN
+F 2 "pad:R_0603_nodraw" V 7030 1800 30  0001 C CNN
 F 3 "" H 7100 1800 30  0000 C CNN
 	1    7100 1800
@@
 F 0 "R10" V 7930 4950 50  0000 C CNN
 F 1 "R" V 7850 4950 50  0000 C CNN
-F 2 "Resistors_SMD:R_0603_HandSoldering" V 7780 4950 30  0001 C CNN
+F 2 "pad:R_0603_nodraw" V 7780 4950 30  0001 C CNN
 F 3 "" H 7850 4950 30  0000 C CNN
 	1    7850 4950
@@
 F 0 "R9" V 7080 4750 50  0000 C CNN
 F 1 "R" V 7000 4750 50  0000 C CNN
-F 2 "Resistors_SMD:R_0603_HandSoldering" V 6930 4750 30  0001 C CNN
+F 2 "pad:R_0603_nodraw" V 6930 4750 30  0001 C CNN
 F 3 "" H 7000 4750 30  0000 C CNN
 	1    7000 4750
@@
 F 0 "R7" V 6780 4400 50  0000 C CNN
 F 1 "R" V 6700 4400 50  0000 C CNN
-F 2 "Resistors_SMD:R_0603_HandSoldering" V 6630 4400 30  0001 C CNN
+F 2 "pad:R_0603_nodraw" V 6630 4400 30  0001 C CNN
 F 3 "" H 6700 4400 30  0000 C CNN
 	1    6700 4400
@@
 F 0 "R6" V 6780 4200 50  0000 C CNN
 F 1 "R" V 6700 4200 50  0000 C CNN
-F 2 "Resistors_SMD:R_0603_HandSoldering" V 6630 4200 30  0001 C CNN
+F 2 "pad:R_0603_nodraw" V 6630 4200 30  0001 C CNN
 F 3 "" H 6700 4200 30  0000 C CNN
 	1    6700 4200
@@
 F 0 "R8" V 7080 3850 50  0000 C CNN
 F 1 "R" V 7000 3850 50  0000 C CNN
-F 2 "Resistors_SMD:R_0603_HandSoldering" V 6930 3850 30  0001 C CNN
+F 2 "pad:R_0603_nodraw" V 6930 3850 30  0001 C CNN
 F 3 "" H 7000 3850 30  0000 C CNN
 	1    7000 3850
@@
 F 0 "R11" V 7380 3250 50  0000 C CNN
 F 1 "R" V 7300 3250 50  0000 C CNN
-F 2 "Resistors_SMD:R_0603_HandSoldering" V 7230 3250 30  0001 C CNN
+F 2 "pad:R_0603_nodraw" V 7230 3250 30  0001 C CNN
 F 3 "" H 7300 3250 30  0000 C CNN
 	1    7300 3250
@@
 F 0 "R12" V 7480 5300 50  0000 C CNN
 F 1 "R" V 7400 5300 50  0000 C CNN
-F 2 "Resistors_SMD:R_0603_HandSoldering" V 7330 5300 30  0001 C CNN
+F 2 "pad:R_0603_nodraw" V 7330 5300 30  0001 C CNN
 F 3 "" H 7400 5300 30  0000 C CNN
 	1    7400 5300
